File: kicad/bno085/slime.kicad_sch (KiCad schematic)
At the start: 39 parts, among them J1 USB4125-GF-A_REVA, J2 Conn_02x03_Odd_Even, J3 Conn_01x05, J4 Conn_01x02, SW1 SW_SPDT, U1 MCP73832-2-OT, U2 BQ297xy, U3 CSD85302L, U4 NCP177BMX330TCG, U5 ASAK-32.7680KHZ-LRS-T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

Commit message: updated titel block
Other:
- title: (none) -> slime_minimax with bno085
Changed lines of the file:
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@@
 (kicad_sch (version 20211123) (generator eeschema)
   (paper "A4")
+  (title_block
+    (title "slime_minimax with bno085")
+    (date "2022-11-16")
+    (rev "c")
+  )
   (junction (at 29.21 73.66) (diameter 0) (color 0 0 0 0)
   )
