File: kicad/bno055/bno055.kicad_sch (KiCad schematic)
At the start: 37 parts, among them J1 USB4125-GF-A_REVA, J2 Conn_02x03_Odd_Even, J3 Conn_01x05, J4 Conn_01x02, SW1 SW_SPDT, U1 MCP73832-2-OT, U2 BQ297xy, U3 CSD85302L, U4 NCP177BMX330TCG, U5 BMI160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

Commit message: added bno055 support unfortunately some componts ha to be mouted on the back as they were to lage for the front
Parts:
- removed U5: BMI160, Package_LGA:Bosch_LGA-14_3x2.5mm_P0.5mm, symbol Sensor_Motion:BMI160
- added C10, C11: 15pf, Capacitor_SMD:C_0402_1005Metric, symbol Device:C
- added C9: 100nf, Capacitor_SMD:C_0402_1005Metric, symbol Device:C
- added R13: 10k, Resistor_SMD:R_0402_1005Metric, symbol Device:R
- added U5: BNO055, Package_LGA:LGA-28_5.2x3.8mm_P0.5mm, symbol Sensor_Motion:BNO055
- added Y1: MC-405 32.0000K-R3: PURE SN, Crystal:Crystal_SMD_SeikoEpson_MC405-2Pin_9.6x4.1mm, symbol Device:Crystal
Connections:
- net MOSI is gone; now on net ADDRESS: J3.5 (Pin_5)
- net +3.3V: now also R13.2, U5.28 (VDDIO), U5.3 (VDD)
- net ADDRESS: now also U5.17 (COM3)
- net BOOTN: now also R13.1, U5.4 (~{BOOT_LOAD_PIN})
- net GND: now also C10.2, C11.2, C9.2, U5.10 (BL_IND), U5.15 (GNDIO), U5.16 (GNDIO), U5.18 (COM2), U5.2 (GND), U5.25 (GNDIO), U5.5 (PS1), U5.6 (PS0)
- net H_SCL: now also U5.19 (COM1)
- net H_SDA: now also U5.20 (COM0)
- net INT: now also U5.14 (INT)
- net RESET: now also U5.11 (~{RESET})
- new net: C10.1, U5.26 (XOUT32), Y1.2
- new net: C11.1, U5.27 (XIN32), Y1.1
- new net cap: C9.1, U5.9 (CAP)
- no-connect marks 14 -> 8
Other:
- note added: "BNO055"
- note removed: "BMI160"
- title: slime_minimax with bmi160 -> slime_minimax with bno055
- moved on the sheet: JP1, R15, R16
