File: kicad/mpu9250/mpu9250.kicad_pcb (KiCad board)
At the start: 2 copper layers, 31 x 42 mm, 39 parts, among them J1 USB4125-GF-A_REVA, J2 PinHeader_2x03_P2.54mm_Vertic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, J3 PinHeader_1x05_P2.54mm_Vertic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, J4 PinHeader_1x02_P2.54mm_Vertic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, SW1 SW_SPDT, U1 dfn-8_wide, U2 BQ297xy, U3 CSD85302L, U4 NCP177BMX330TCG, U5 BMI160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

Commit message: added support for mpu9250
Parts:
- removed C6: 100nf, Capacitor_SMD:C_0402_1005Metric
- added C10: 100nf, Capacitor_SMD:C_0402_1005Metric, F.Cu at (127.2, 95.2)
- added C9: 100nf, Capacitor_SMD:C_0402_1005Metric, F.Cu at (129.0, 92.4)
- U5: value BMI160 -> mpu9250; footprint Package_LGA:Bosch_LGA-14_3x2.5mm_P0.5mm -> Package_DFN_QFN:QFN-24-1EP_3x3mm_P0.4mm_EP1.75x1.6mm
- moved C7 6.41 mm to (126.6, 89.6), turned to 180 degrees
- moved U5 1.34 mm to (126.2, 92.4)
Connections:
- R12 pad 1: /GPIO0 -> +3.3V
- R12 pad 2: +3.3V -> /GPIO0
- R2 pad 1: +BATT -> /BAT_SENCE
- R2 pad 2: /BAT_SENCE -> +BATT
- U4 pad 5: (no net) -> GND
- U5 pad 1: /ADDRESS -> +3.3V
- U5 pad 10: unconnected-(U5-Pad10) -> Net-(C10-Pad2)
- U5 pad 11: unconnected-(U5-Pad11) -> GND
- U5 pad 12: +3.3V -> unconnected-(U5-Pad12)
- U5 pad 13: /H_SCL -> +3.3V
- U5 pad 14: /H_SDA -> unconnected-(U5-Pad14)
- U5 pad 5: +3.3V -> unconnected-(U5-Pad5)
- U5 pad 6: GND -> unconnected-(U5-Pad6)
- U5 pad 7: GND -> unconnected-(U5-Pad7)
- U5 pad 9: unconnected-(U5-Pad9) -> /ADDRESS
Routing:
- net +3.3V: track 112.8 -> 131.2 mm, vias 7 -> 8
- net /ADDRESS: track 22.6 -> 29.1 mm
- net GND: track 130.3 -> 135.5 mm
- net Net-(R10-Pad1): track 2.33 -> 0.00 mm
- net /GPIO16: track 0.00 -> 2.33 mm
- net /H_SCL: track 34.9 -> 33.2 mm
- net /H_SDA: track 25.2 -> 23.5 mm
- net CH_PROG: track 1.47 -> 0.00 mm
- net /CH_PROG: track 0.00 -> 1.47 mm
- net Net-(C10-Pad2): track 0.00 -> 1.43 mm
- removed copper zone on B.Cu, net GND
- removed copper zone on F.Cu, net GND
Other:
- board text removed: "BMI ADDRESS"
- board text removed: "BMI MODULE"
- board text removed: "BMI PINS"
